File: combo/dumbpad.brd (EAGLE design)
At the start: 97 x 78.5 mm, 45 parts

Commit message: fixing bad merge
Parts:
- removed LOGO3: OSHW-LOGOL, SparkFun-Aesthetics:OSHW-LOGO-L
- moved LOGO2 0.45 mm to (10.1, 59.5), flipped to the top
Connections:
- net N$12: now also S15.S1; no longer S15.S1_0
- net N$13: now also S14.S1; no longer S14.S1_0
- net N$16: now also S12.S1; no longer S12.S1_0
- net N$17: now also S11.S1; no longer S11.S1_0
- net N$18: now also S10.S1; no longer S10.S1_0
- net N$19: now also S9.S1; no longer S9.S1_0
- net N$2: now also S3.S1; no longer S3.S1_0
- net N$3: now also S2.S1; no longer S2.S1_0
- net N$6: now also S8.S1; no longer S8.S1_0
- net N$7: now also S7.S1; no longer S7.S1_0
- net N$8: now also S6.S1; no longer S6.S1_0
- net N$9: now also S5.S1; no longer S5.S1_0
Changed lines of the file:
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@@
 <attribute name="VALUE" x="19.779" y="8.818" size="0.6096" layer="21" rot="R90"/>
 </element>
-<element name="LOGO2" library="SparkFun-Aesthetics" package="OSHW-LOGO-L" value="OSHW-LOGOL" x="10.5" y="59.5" smashed="yes" rot="MR0"/>
-<element name="LOGO3" library="SparkFun-Aesthetics" package="OSHW-LOGO-L" value="OSHW-LOGOL" x="10.5" y="59.5" smashed="yes"/>
 </elements>
 <signals>
@@
 </signal>
 <signal name="N$2">
-<contactref element="S3" pad="S1_0"/>
+<contactref element="S3" pad="S1"/>
 <contactref element="D3" pad="A"/>
 <wire x1="71.91" y1="65.46" x2="73.18" y2="64.19" width="0.1524" layer="1"/>
@@
 </signal>
 <signal name="N$3">
-<contactref element="S2" pad="S1_0"/>
+<contactref element="S2" pad="S1"/>
 <contactref element="D2" pad="A"/>
 <wire x1="52.86" y1="65.46" x2="54.13" y2="64.19" width="0.1524" layer="1"/>
@@
 </signal>
 <signal name="N$6">
-<contactref element="S8" pad="S1_0"/>
+<contactref element="S8" pad="S1"/>
 <contactref element="D8" pad="A"/>
 <wire x1="90.96" y1="46.41" x2="92.23" y2="45.14" width="0.1524" layer="1"/>
@@
 </signal>
 <signal name="N$7">
-<contactref element="S7" pad="S1_0"/>
+<contactref element="S7" pad="S1"/>
 <contactref element="D7" pad="A"/>
 <wire x1="71.91" y1="46.41" x2="73.18" y2="45.14" width="0.1524" layer="1"/>
@@
 </signal>
 <signal name="N$8">
-<contactref element="S6" pad="S1_0"/>
+<contactref element="S6" pad="S1"/>
 <contactref element="D6" pad="A"/>
 <wire x1="52.86" y1="46.41" x2="54.13" y2="45.14" width="0.1524" layer="1"/>
@@
 </signal>
 <signal name="N$9">
-<contactref element="S5" pad="S1_0"/>
+<contactref element="S5" pad="S1"/>
 <contactref element="D5" pad="A"/>
 <wire x1="33.81" y1="46.41" x2="35.08" y2="45.14" width="0.1524" layer="1"/>
@@
 </signal>
 <signal name="N$12">
-<contactref element="S15" pad="S1_0"/>
+<contactref element="S15" pad="S1"/>
 <contactref element="D15" pad="A"/>
 <wire x1="71.91" y1="8.31" x2="73.18" y2="7.04" width="0.1524" layer="1"/>
@@
 </signal>
 <signal name="N$13">
-<contactref element="S14" pad="S1_0"/>
+<contactref element="S14" pad="S1"/>
 <contactref element="D14" pad="A"/>
 <wire x1="52.86" y1="8.31" x2="54.13" y2="7.04" width="0.1524" layer="1"/>
@@
 </signal>
 <signal name="N$16">
-<contactref element="S12" pad="S1_0"/>
+<contactref element="S12" pad="S1"/>
 <contactref element="D12" pad="A"/>
 <wire x1="90.96" y1="27.36" x2="92.23" y2="26.09" width="0.1524" layer="1"/>
@@
 </signal>
 <signal name="N$17">
-<contactref element="S11" pad="S1_0"/>
+<contactref element="S11" pad="S1"/>
 <contactref element="D11" pad="A"/>
 <wire x1="71.91" y1="27.36" x2="73.18" y2="26.09" width="0.1524" layer="1"/>
@@
 </signal>
 <signal name="N$18">
-<contactref element="S10" pad="S1_0"/>
+<contactref element="S10" pad="S1"/>
 <contactref element="D10" pad="A"/>
 <wire x1="52.86" y1="27.36" x2="54.13" y2="26.09" width="0.1524" layer="1"/>
@@
 </signal>
 <signal name="N$19">
-<contactref element="S9" pad="S1_0"/>
+<contactref element="S9" pad="S1"/>
 <contactref element="D9" pad="A"/>
 <wire x1="33.81" y1="27.36" x2="35.08" y2="26.09" width="0.1524" layer="1"/>

Commit message: fixing naming issue in combo
Connections:
- net LED0: now also B1.13, R3.P$2; no longer B1.15, R1.P$2
- net LED2: now also B1.15, R1.P$2; no longer B1.13, R3.P$2
Routing:
- net LED2: track 21.2 -> 19.2 mm
- net LED0: track 19.2 -> 21.2 mm
Changed lines of the file:
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@@
 </signal>
 <signal name="LED0">
-<contactref element="R1" pad="P$2"/>
-<contactref element="B1" pad="15"/>
-<wire x1="13.86" y1="34.25" x2="16.25" y2="34.25" width="0.1524" layer="1"/>
-<wire x1="19" y1="48.01" x2="17.67" y2="49.34" width="0.1524" layer="1"/>
-<wire x1="16.25" y1="34.25" x2="19" y2="37" width="0.1524" layer="1"/>
-<wire x1="19" y1="37" x2="19" y2="48.01" width="0.1524" layer="1"/>
+<contactref element="B1" pad="13"/>
+<contactref element="R3" pad="P$2"/>
+<wire x1="13.5" y1="35.75" x2="17" y2="35.75" width="0.1524" layer="1"/>
+<wire x1="17" y1="35.75" x2="18.5" y2="37.25" width="0.1524" layer="1"/>
+<wire x1="18.5" y1="37.25" x2="18.5" y2="43.43" width="0.1524" layer="1"/>
+<wire x1="13.86" y1="28.75" x2="12.25" y2="30.36" width="0.1524" layer="1"/>
+<wire x1="12.25" y1="30.36" x2="12.25" y2="34.5" width="0.1524" layer="1"/>
+<wire x1="12.25" y1="34.5" x2="13.5" y2="35.75" width="0.1524" layer="1"/>
+<wire x1="18.5" y1="43.43" x2="17.67" y2="44.26" width="0.1524" layer="1"/>
 </signal>
 <signal name="LED1">
@@
 </signal>
 <signal name="LED2">
-<contactref element="B1" pad="13"/>
-<contactref element="R3" pad="P$2"/>
-<wire x1="13.5" y1="35.75" x2="17" y2="35.75" width="0.1524" layer="1"/>
-<wire x1="18.5" y1="43.43" x2="17.67" y2="44.26" width="0.1524" layer="1"/>
-<wire x1="17" y1="35.75" x2="18.5" y2="37.25" width="0.1524" layer="1"/>
-<wire x1="18.5" y1="37.25" x2="18.5" y2="43.43" width="0.1524" layer="1"/>
-<wire x1="13.86" y1="28.75" x2="12.25" y2="30.36" width="0.1524" layer="1"/>
-<wire x1="12.25" y1="30.36" x2="12.25" y2="34.5" width="0.1524" layer="1"/>
-<wire x1="12.25" y1="34.5" x2="13.5" y2="35.75" width="0.1524" layer="1"/>
+<contactref element="B1" pad="15"/>
+<contactref element="R1" pad="P$2"/>
+<wire x1="13.86" y1="34.25" x2="16.25" y2="34.25" width="0.1524" layer="1"/>
+<wire x1="16.25" y1="34.25" x2="19" y2="37" width="0.1524" layer="1"/>
+<wire x1="19" y1="37" x2="19" y2="48.01" width="0.1524" layer="1"/>
+<wire x1="19" y1="48.01" x2="17.67" y2="49.34" width="0.1524" layer="1"/>
 </signal>
 <signal name="COL0">

Commit message: fixed encoder pin naming mismatch, updated screenshot
Connections:
- net ENCODER1_L0: now also B1.6, RE_0_4.B, RE_3_4.B; no longer B1.5, RE_0_4.A, RE_3_4.A
- net ENCODER1_L1: now also B1.5, RE_0_4.A, RE_3_4.A; no longer B1.6, RE_0_4.B, RE_3_4.B
Routing:
- net ENCODER1_L1: track 160.3 -> 157.7 mm
- net ENCODER1_L0: track 157.7 -> 160.3 mm
Changed lines of the file:
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@@
 <wire x1="14.31" y1="31.5" x2="19.5" y2="36.69" width="0.1524" layer="1"/>
 </signal>
-<signal name="ENCODER1_L0">
+<signal name="ENCODER1_L1">
 <contactref element="B1" pad="5"/>
 <contactref element="RE_3_4" pad="A"/>
@@
 <wire x1="19.75" y1="77.75" x2="4.04" y2="62.04" width="0.1524" layer="1"/>
 </signal>
-<signal name="ENCODER1_L1">
+<signal name="ENCODER1_L0">
 <contactref element="B1" pad="6"/>
 <contactref element="RE_3_4" pad="B"/>
