File: combo_oled/dumbpad.kicad_sch (KiCad schematic)
At the start: 43 parts, among them J1 Conn_01x04_Female, J2 Conn_01x04_Female

Commit message: fix schematic and remove missing drawing sheet
Connections:
- net ENCODER0_L0: now also RE_0_1.B, RE_3_0.B, RE_3_1.B
- net ENCODER0_L1: now also RE_0_1.A, RE_3_0.A, RE_3_1.A
- net ENCODER1_L0: now also RE_0_4.B, RE_3_4.B
- net ENCODER1_L1: now also RE_0_4.A, RE_3_4.A
- net GND: now also RE_0_1.C, RE_0_4.C, RE_3_0.C, RE_3_1.C, RE_3_4.C
